File: hexboard.kicad_pcb (KiCad board)
At the start: 2 copper layers, 306.7 x 107.3 mm, 158 parts, among them SW1 SW_Push, U1 Teensy2.0_(C)

Commit message: dunno whative changed whatever
Parts:
- removed LED1: CAPS/1, Keebio:MX_LED
- removed LED2: SCROLL/2, Keebio:MX_LED
- removed LED3: NUM/3, Keebio:MX_LED
- removed LED4: 4, Keebio:MX_LED
- removed R1: R, Keebio:Resistor-Hybrid
- removed the REF** at (87.0, 52.7)
- removed the REF** at (66.0, 83.2)
- removed the REF** at (288.9, 57.1)
- removed the REF** at (303.5, 125.1)
- removed the REF** at (234.3, 144.1)
- removed the REF** at (172.7, 144.1)
- removed the REF** at (79.4, 125.1)
- removed e: MountingHole_3.2mm_M3_Pad_Via, MountingHole:MountingHole_3.2mm_M3_Pad_Via
- added REF**: Symbol_CC-ShareAlike_CopperTop_Small, Symbol:Symbol_CC-ShareAlike_CopperTop_Small, F.Cu at (247.0, 150.5)
- added REF**: Symbol_CC-Attribution_CopperTop_Small, Symbol:Symbol_CC-Attribution_CopperTop_Small, F.Cu at (240.7, 150.5)
- added REF**: OSHW-Logo2_7.3x6mm_Copper, Symbol:OSHW-Logo2_7.3x6mm_Copper, F.Cu at (233.7, 150.5)
- added REF**: KiCad-Logo2_5mm_Copper, Symbol:KiCad-Logo2_5mm_Copper, F.Cu at (222.2, 149.9)
- added U4: HOLE, Keebio:MountingHole, F.Cu at (36.2, 156.8)
- added U4: HOLE, Keebio:MountingHole, F.Cu at (348.0, 156.8)
- added U4: HOLE, Keebio:MountingHole, F.Cu at (348.0, 54.6)
- added U4: HOLE, Keebio:MountingHole, F.Cu at (36.2, 54.6)
- added U4: HOLE, Keebio:MountingHole, F.Cu at (192.1, 156.8)
- added U4: HOLE, Keebio:MountingHole, F.Cu at (192.1, 54.6)
- moved SW1 34.9 mm to (66.0, 88.9), turned to 270 degrees
- moved U1 18.7 mm to (67.9, 64.8)
- moved D6 0.63 mm to (68.3, 76.2)
Routing:
- net Net-(U1-Pad18): track 304.0 -> 0.00 mm
- net Net-(U1-Pad19): track 301.2 -> 0.00 mm
- net Net-(U1-Pad20): track 300.8 -> 0.00 mm
- net Net-(U1-Pad21): track 294.8 -> 0.00 mm
- net Net-(SW1-Pad2): track 40.7 -> 14.4 mm, vias 1 -> 0
- net Net-(LED1-Pad1): track 22.9 -> 0.00 mm
- net /col3: track 150.1 -> 127.7 mm
- net /col4: track 149.7 -> 128.4 mm
- net /col7: track 191.4 -> 170.5 mm
- net /col5: track 153.5 -> 133.7 mm
- net /col6: track 155.1 -> 135.6 mm
- net /col8: track 216.4 -> 197.6 mm
- net /col14: track 360.0 -> 341.3 mm
- net /col10: track 232.6 -> 214.1 mm
- net /col12: track 289.0 -> 270.5 mm
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Other:
- board size 306.7 x 107.3 mm -> 321.9 x 112.4 mm
- net class Default: trace_width 0.2032 -> 0.3048
- board text added: "HexBoard"
- board text added: "LO"
- board text added: "Mk.I"
- board text added: "VE"
- board text added: "by @Hexadecimaaal"
- board text added: "made with"
