File: hexboard.sch (KiCad schematic (older format))
At the start: 150 parts, among them SW1 SW_Push, U1 Teensy2.0_(C)

Commit message: dunno whative changed whatever
Parts:
- removed LED1: CAPS/1, Keebio:MX_LED, symbol Device:LED_Small
- removed LED2: SCROLL/2, Keebio:MX_LED, symbol Device:LED_Small
- removed LED3: NUM/3, Keebio:MX_LED, symbol Device:LED_Small
- removed LED4: 4, Keebio:MX_LED, symbol Device:LED_Small
- removed R1: R, Keebio:Resistor-Hybrid, symbol Device:R_Small
Changed lines of the file:
@@
-$EndComp
-$Comp
-L MX_Alps_Hybrid:MX-NoLED MX72
-U 1 1 5EF86E20
-P 6100 2900
-F 0 "MX72" H 6133 3123 60  0000 C CNN
-F 1 "MX-NoLED" H 6133 3049 20  0000 C CNN
-F 2 "MX Only:MXOnly-1.5U-Vertical-NoLED" H 5475 2875 60  0001 C CNN
-F 3 "" H 5475 2875 60  0001 C CNN
-	1    6100 2900
-	1    0    0    -1
 $EndComp
 $Comp
@@
 	1850 4450 1850 5050
 $Comp
-L power:GND #PWR01
-U 1 1 5F4A8645
-P 10700 4500
-F 0 "#PWR01" H 10700 4250 50  0001 C CNN
-F 1 "GND" H 10705 4327 50  0000 C CNN
-F 2 "" H 10700 4500 50  0001 C CNN
-F 3 "" H 10700 4500 50  0001 C CNN
-	1    10700 4500
-	1    0    0    -1
-$EndComp
-$Comp
-L Device:LED_Small LED1
-U 1 1 5F4B34FC
-P 10600 3700
-F 0 "LED1" H 10750 3650 50  0000 C CNN
-F 1 "CAPS/1" H 10300 3700 50  0000 C CNN
-F 2 "Keebio:MX_LED" V 10600 3700 50  0001 C CNN
-F 3 "~" V 10600 3700 50  0001 C CNN
-	1    10600 3700
-	-1   0    0    1
-$EndComp
-$Comp
-L Device:LED_Small LED2
-U 1 1 5F4B4D59
-P 10600 3800
-F 0 "LED2" H 10750 3750 50  0000 C CNN
-F 1 "SCROLL/2" H 10300 3800 50  0000 C CNN
-F 2 "Keebio:MX_LED" V 10600 3800 50  0001 C CNN
-F 3 "~" V 10600 3800 50  0001 C CNN
-	1    10600 3800
-	-1   0    0    1
-$EndComp
-$Comp
-L Device:LED_Small LED3
-U 1 1 5F4B6BA9
-P 10600 3900
-F 0 "LED3" H 10750 3850 50  0000 C CNN
-F 1 "NUM/3" H 10300 3900 50  0000 C CNN
-F 2 "Keebio:MX_LED" V 10600 3900 50  0001 C CNN
-F 3 "~" V 10600 3900 50  0001 C CNN
-	1    10600 3900
-	-1   0    0    1
-$EndComp
-$Comp
-L Device:LED_Small LED4
-U 1 1 5F4B7386
-P 10600 4000
-F 0 "LED4" H 10750 3950 50  0000 C CNN
-F 1 "4" H 10300 4000 50  0000 C CNN
-F 2 "Keebio:MX_LED" V 10600 4000 50  0001 C CNN
-F 3 "~" V 10600 4000 50  0001 C CNN
-	1    10600 4000
-	-1   0    0    1
-$EndComp
-Wire Wire Line
-	10700 3700 10700 3800
-Connection ~ 10700 3800
-Wire Wire Line
-	10700 3800 10700 3900
-Connection ~ 10700 3900
-Wire Wire Line
-	10700 3900 10700 4000
-Wire Wire Line
-	10400 3700 10500 3700
-Wire Wire Line
-	10400 3800 10500 3800
-Wire Wire Line
-	10400 3900 10500 3900
-Wire Wire Line
-	10400 4000 10500 4000
-$Comp
-L Device:R_Small R1
-U 1 1 5F54F79E
-P 10700 4300
-F 0 "R1" H 10759 4346 50  0000 L CNN
-F 1 "R" H 10759 4255 50  0000 L CNN
-F 2 "Keebio:Resistor-Hybrid" H 10700 4300 50  0001 C CNN
-F 3 "~" H 10700 4300 50  0001 C CNN
-	1    10700 4300
-	1    0    0    -1
-$EndComp
-Wire Wire Line
-	10700 4400 10700 4500
-Wire Wire Line
-	10700 4200 10700 4000
-Connection ~ 10700 4000
+L MX_Alps_Hybrid:MX-NoLED MX72
+U 1 1 5EF86E20
+P 6100 2900
+F 0 "MX72" H 6133 3123 60  0000 C CNN
+F 1 "MX-NoLED" H 6133 3049 20  0000 C CNN
+F 2 "MX Only:MXOnly-1.5U-Vertical-NoLED" H 5475 2875 60  0001 C CNN
+F 3 "" H 5475 2875 60  0001 C CNN
+	1    6100 2900
+	1    0    0    -1
+$EndComp
 $EndSCHEMATC
